Commit message: Update MyRobot locomotion training config

File: Huazhong1/urdf/Huazhong1.urdf (robot description, URDF)
Before this commit: robot Huazhong1, 13 links, 12 joints
Links:
- link Left_knee_pitch_link: geometry collision box size=0.10 0.10 0.3; visual mesh filename=../meshes/Left_knee_pitch_link.STL
- link Right_knee_pitch_link: geometry collision box size=0.10 0.10 0.3; visual mesh filename=../meshes/Right_knee_pitch_link.STL
Joints:
- joint Left_knee_pitch_joint: limit lower=0.0873 upper=2.1817 effort=1000 velocity=20 -> lower=0.0873 upper=1.7453 effort=1000 velocity=20
- joint Left_leg_roll_joint: limit lower=-0.5236 upper=0.5236 effort=1000 velocity=20 -> lower=-0.0349 upper=0.5236 effort=1000 velocity=20
- joint Left_leg_yaw_joint: axis 0 0 1 -> (none); limit lower=-0.1745 upper=0.6981 effort=1000 velocity=20 -> (none); type revolute -> fixed
- joint Right_knee_pitch_joint: limit lower=0.0873 upper=2.1817 effort=1000 velocity=20 -> lower=0.0873 upper=1.7453 effort=1000 velocity=20
- joint Right_leg_roll_joint: limit lower=-0.5236 upper=0.5236 effort=1000 velocity=20 -> lower=-0.5236 upper=0.0349 effort=1000 velocity=20
- joint Right_leg_yaw_joint: axis 0 0 1 -> (none); limit lower=-0.6981 upper=0.1745 effort=1000 velocity=20 -> (none); type revolute -> fixed
